Commit message: Use the weighed masses for the own mecanum robot
The robot was weighed: 1927.4 g for the body without wheels and 51.65 g
per wheel, 2.134 kg in total (the URDF had guesses totalling 3.0 kg).
Every component is assumed homogeneous:

- base_link: uniform density over chassis_visual.stl. The CoM moves to
  the mesh centroid, (-1.1, 0.1, -19.7) mm instead of the hand-set
  16 mm forward offset.
- each wheel: one density over the hub cylinder and the 9 rollers, so
  the mass is split by volume (hub 32.59 g, roller 2.118 g). Roller
  inertia now comes from the barrel mesh instead of a cylinder.

docs/analysis/set_masses.py computes and writes the <inertial> blocks;
re-run it after copying a newer robot.urdf from Mecanum-TDK. The MPC
reads the new parameters from the URDF (m_e 3.17 -> 2.21 kg).

Co-Authored-By: Claude Opus 5.5 <noreply@anthropic.com>

File: tb3_sim_bringup/models/own_mecanum/robot.urdf (robot description, URDF)
Before this commit: robot mecanum_rollers, 41 links, 40 joints
Links:
- link base_link: mass 2.6 -> 1.9274
- link front_left_roller_00: mass 0.005 -> 0.00211808
- link front_left_roller_01: mass 0.005 -> 0.00211808
- link front_left_roller_02: mass 0.005 -> 0.00211808
- link front_left_roller_03: mass 0.005 -> 0.00211808
- link front_left_roller_04: mass 0.005 -> 0.00211808
- link front_left_roller_05: mass 0.005 -> 0.00211808
- link front_left_roller_06: mass 0.005 -> 0.00211808
- link front_left_roller_07: mass 0.005 -> 0.00211808
- link front_left_roller_08: mass 0.005 -> 0.00211808
- link front_left_wheel: mass 0.055 -> 0.0325873
- link front_right_roller_00: mass 0.005 -> 0.00211808
- link front_right_roller_01: mass 0.005 -> 0.00211808
- link front_right_roller_02: mass 0.005 -> 0.00211808
- link front_right_roller_03: mass 0.005 -> 0.00211808
- link front_right_roller_04: mass 0.005 -> 0.00211808
- link front_right_roller_05: mass 0.005 -> 0.00211808
- link front_right_roller_06: mass 0.005 -> 0.00211808
- link front_right_roller_07: mass 0.005 -> 0.00211808
- link front_right_roller_08: mass 0.005 -> 0.00211808
- link front_right_wheel: mass 0.055 -> 0.0325873
- link rear_left_roller_00: mass 0.005 -> 0.00211808
- link rear_left_roller_01: mass 0.005 -> 0.00211808
- link rear_left_roller_02: mass 0.005 -> 0.00211808
- link rear_left_roller_03: mass 0.005 -> 0.00211808
- link rear_left_roller_04: mass 0.005 -> 0.00211808
- link rear_left_roller_05: mass 0.005 -> 0.00211808
- link rear_left_roller_06: mass 0.005 -> 0.00211808
- link rear_left_roller_07: mass 0.005 -> 0.00211808
- link rear_left_roller_08: mass 0.005 -> 0.00211808
- link rear_left_wheel: mass 0.055 -> 0.0325873
- link rear_right_roller_00: mass 0.005 -> 0.00211808
- link rear_right_roller_01: mass 0.005 -> 0.00211808
- link rear_right_roller_02: mass 0.005 -> 0.00211808
- link rear_right_roller_03: mass 0.005 -> 0.00211808
- link rear_right_roller_04: mass 0.005 -> 0.00211808
- link rear_right_roller_05: mass 0.005 -> 0.00211808
- link rear_right_roller_06: mass 0.005 -> 0.00211808
- link rear_right_roller_07: mass 0.005 -> 0.00211808
- link rear_right_roller_08: mass 0.005 -> 0.00211808
- link rear_right_wheel: mass 0.055 -> 0.0325873

File: tb3_sim_bringup/urdf/own_mecanum.urdf.xacro (robot description, xacro)
@@ -2,6 +2,8 @@
 <!--
   Own mecanum robot (github.com/Kemenylegeny/Mecanum-TDK, assets/robots/own_mecanum) for gz sim.
-  models/own_mecanum/robot.urdf + meshes/ are copied from that repo UNCHANGED, so a newer
-  version can be dropped in over them. Everything the simulation needs on top of it lives here:
+  models/own_mecanum/robot.urdf + meshes/ are copied from that repo. The only local change is
+  the <inertial> blocks: weighed masses (body 1927.4 g, wheel 51.65 g), homogeneous components,
+  written by docs/analysis/set_masses.py. To update the robot, drop a newer robot.urdf in and
+  re-run that script with its write option. Everything the simulation needs on top of it lives here:
   base_footprint, lidar + IMU frames and sensors, roller friction, the MecanumDrive and
   JointStatePublisher systems. The launch file rewrites the URDF's relative mesh paths
